File: ak-tracker/ak-tracker.kicad_sch (KiCad schematic)
At the start: 13 parts, among them J1 left, J2 right, SW2 Reset, SW3 SW_DIP_x02, U1 BMA400, U2 TPL5010

Commit message: 3k3 & silk screen
Parts:
- SW3: value SW_DIP_x02 -> Wd Acc
Changed lines of the file:
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@@
 			)
 		)
-		(property "Value" "SW_DIP_x02"
+		(property "Value" "Wd Acc"
 			(at 138.43 92.71 0)
 			(show_name no)
