File: power-board/power-board.kicad_sch (KiCad schematic)
At the start: 0 parts

Commit message: power board diagram
Parts:
- added BT1: 18650, TerminalBlock_Phoenix:TerminalBlock_Phoenix_PT-1,5-2-5.0-H_1x02_P5.00mm_Horizontal, symbol Device:Battery_Cell
- added C1: 100n, Capacitor_SMD:C_0805_2012Metric_Pad1.18x1.45mm_HandSolder, symbol Device:C
- added C2: 1n/50V, Capacitor_SMD:C_0805_2012Metric_Pad1.18x1.45mm_HandSolder, symbol Device:C
- added C3, C4: 4u7, Capacitor_SMD:C_0805_2012Metric_Pad1.18x1.45mm_HandSolder, symbol Device:C
- added C5: 1u, Capacitor_SMD:C_0805_2012Metric_Pad1.18x1.45mm_HandSolder, symbol Device:C
- added C6: 10u, Capacitor_SMD:C_0805_2012Metric_Pad1.18x1.45mm_HandSolder, symbol Device:C
- added C7, C8: 1000u, Capacitor_THT:CP_Radial_D12.5mm_P5.00mm, symbol Device:C_Polarized
- added F1: 2A slow, Fuse:Fuseholder_Cylinder-5x20mm_Schurter_0031_8201_Horizontal_Open, symbol Device:Fuse
- added J1: USB_C, Connector_USB:USB_C_Receptacle_GCT_USB4125-xx-x-0190_6P_TopMnt_Horizontal, symbol Connector:USB_C_Receptacle_PowerOnly_6P
- added J2, J3, J4: Conn_01x02, TerminalBlock_Phoenix:TerminalBlock_Phoenix_PT-1,5-2-5.0-H_1x02_P5.00mm_Horizontal, symbol Connector_Generic:Conn_01x02
- added J6: Conn_01x03, TerminalBlock_Phoenix:TerminalBlock_Phoenix_PT-1,5-3-3.5-H_1x03_P3.50mm_Horizontal, symbol Connector_Generic:Conn_01x03
- added Q1, Q2: AOB2146L, Package_TO_SOT_SMD:TO-263-2, symbol Transistor_FET:IRFS4115
- added R1: 330, Resistor_SMD:R_0805_2012Metric_Pad1.20x1.40mm_HandSolder, symbol Device:R
- added R10, R9: 5k1, Resistor_SMD:R_0805_2012Metric_Pad1.20x1.40mm_HandSolder, symbol Device:R
- added R2: 2k7, Resistor_SMD:R_0805_2012Metric_Pad1.20x1.40mm_HandSolder, symbol Device:R
- added R3: 1k, Resistor_SMD:R_0805_2012Metric_Pad1.20x1.40mm_HandSolder, symbol Device:R
- added R4: 3k3, Resistor_SMD:R_0805_2012Metric_Pad1.20x1.40mm_HandSolder, symbol Device:R
- added R5: 10k, Resistor_SMD:R_0805_2012Metric_Pad1.20x1.40mm_HandSolder, symbol Device:R
- added R6: 100k, Resistor_SMD:R_0805_2012Metric_Pad1.20x1.40mm_HandSolder, symbol Device:R
- added R7: LDR03, OptoDevice:R_LDR_10x8.5mm_P7.6mm_Vertical, symbol Sensor_Optical:LDR03
- added R8: 470, Resistor_SMD:R_0805_2012Metric_Pad1.20x1.40mm_HandSolder, symbol Device:R
- added SW1: On, symbol Switch:SW_SPST
- added SW2: Mode, symbol Switch:SW_SPST
- added U1: AP9101CK6, Package_TO_SOT_SMD:SOT-23-6, symbol Battery_Management:AP9101CK6
- added U2: AP130-33Y, Package_TO_SOT_SMD:SOT-89-3, symbol Regulator_Linear:AP130-33Y
- added U3: MCP73831-3-OT, Package_TO_SOT_SMD:SOT-23-5, symbol Battery_Management:MCP73831-3-OT
- added U4: ESP8266-NodeM, RF_Module:ESP32-C3-DevKitM-1, symbol rgb_matrix:ESP8266-NodeM
Connections:
- new net: J1.B5 (CC2), R9.1
- new net: C4.1, F1.1, R1.1, SW1.1 (A), U3.3 (V_{BAT})
- new net: BT1.1 (+), F1.2
- new net: Q2.1 (G), U1.3 (CO)
- new net: Q1.2 (D), Q2.2 (D)
- new net: Q1.1 (G), U1.1 (DO)
- new net: R6.1, R7.2, U4.16 (A0)
- new net: J1.A5 (CC1), R10.1
- new net: C2.1, J1.SH (SHIELD), R3.2
- new net: R4.1, U3.5 (PROG)
- new net: C1.1, R1.2, U1.5 (VDD)
- new net: C3.1, J1.A9 (VBUS), J1.B9 (VBUS), U3.4 (V_{DD})
- new net: R2.1, U1.2 (VM)
- new net: R5.2, SW2.2 (B), U4.14 (D1)
- new net: J6.2 (Pin_2), R8.1
- new net: R8.2, U4.13 (D2)
- new net +3V3: C6.1, C7.1, R5.1, R7.1, U2.1 (VO), U4.1 (3V3), U4.10 (3V3), U4.26 (3V3)
- new net +VSW: C5.1, C8.1, J2.1 (Pin_1), J3.1 (Pin_1), J4.1 (Pin_1), J6.1 (Pin_1), SW1.2 (B), U2.3 (VI)
- new net BAT-: BT1.2 (-), C1.2, Q2.3 (S), U1.6 (VSS)
- new net GND: C2.2, C3.2, C4.2, C5.2, C6.2, C7.2, C8.2, J1.A12 (GND), J1.B12 (GND), J2.2 (Pin_2), J3.2 (Pin_2), J4.2 (Pin_2), J6.3 (Pin_3), Q1.3 (S), R10.2, R2.2, R3.1, R4.2, R6.2, R9.2, SW2.1 (A), U2.2 (GND), U3.2 (V_{SS}), U4.2 (GND), U4.25 (GND), U4.29 (GND), U4.9 (GND)
- no-connect marks 0 -> 2
Other:
- note added: "Power must be directly connected to all four panels"
- note added: "Should mechanically block USB input when On"
- note added: "star ground"
