File: power-board/power-board.kicad_pcb (KiCad board)
At the start: 2 copper layers, 100 x 100 mm, 46 parts, among them J1 USB_C, J2 - +, J3 + -, J4 + -, J5 Bat+, J6 - In +, J7 Bat-, Q1 AOB2146L, Q2 AOB2146L, Q3 AON7407, SW1 On, SW2 Mode, U1 AP9101CAK6, U2 AP130-33Y, U3 MCP73831-3-OT, U4 ESP8266-NodeM

Commit message: small final adjustment
Parts:
- moved TP6 0.16 mm to (136.6, 139.7)
- moved J3 0.05 mm to (55.1, 145.3)
Routing:
- net +3V3: track 163.2 -> 161.2 mm
Changed lines of the file:
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@@
 	(footprint "Connector_PinHeader_2.54mm:PinHeader_2x01_P2.54mm_Vertical"
 		(layer "F.Cu")
-		(at 55.065 145.4 -90)
+		(at 55.065 145.35 -90)
 		(descr "Through hole straight pin header, 2x01, 2.54mm pitch, double rows")
 		(tags "Through hole pin header THT 2x01 2.54mm double row")
@@
 	(footprint "TestPoint:TestPoint_Pad_2.0x2.0mm"
 		(layer "F.Cu")
-		(at 136.55 139.55)
+		(at 136.6 139.7)
 		(descr "SMD rectangular pad as test Point, square 2.0mm side length")
 		(tags "test point SMD pad rectangle square")
@@
 	)
 	(segment
+		(start 143 53.5)
+		(end 143 65.86)
+		(width 0.2)
+		(layer "F.Cu")
+		(net "+3V3")
+	)
+	(segment
+		(start 113.75 53.25)
+		(end 142.75 53.25)
+		(width 0.2)
+		(layer "F.Cu")
+		(net "+3V3")
+	)
+	(segment
 		(start 140.785 90.935)
 		(end 130.98823 90.935)
@@
 	)
 	(segment
-		(start 111.675 55.325)
-		(end 115.755 51.245)
-		(width 0.2)
-		(layer "F.Cu")
-		(net "+3V3")
-	)
-	(segment
 		(start 117.925 80.775)
 		(end 130.69823 80.775)
@@
 	)
 	(segment
+		(start 111.675 55.53)
+		(end 111.675 55.325)
+		(width 0.2)
+		(layer "F.Cu")
+		(net "+3V3")
+	)
+	(segment
 		(start 138.925 68.075)
 		(end 140.785 68.075)
@@
 	)
 	(segment
-		(start 115.755 51.245)
-		(end 141.245 51.245)
-		(width 0.2)
-		(layer "F.Cu")
-		(net "+3V3")
-	)
-	(segment
-		(start 111.675 55.53)
-		(end 111.675 55.325)
-		(width 0.2)
-		(layer "F.Cu")
-		(net "+3V3")
-	)
-	(segment
 		(start 130.935 128.06177)
 		(end 130.92323 128.05)
@@
 	)
 	(segment
-		(start 143 53)
-		(end 143 65.86)
-		(width 0.2)
-		(layer "F.Cu")
-		(net "+3V3")
-	)
-	(segment
 		(start 130.92323 128.05)
 		(end 140.65 128.05)
@@
 	)
 	(segment
-		(start 141.245 51.245)
-		(end 143 53)
+		(start 143 65.86)
+		(end 140.785 68.075)
 		(width 0.2)
 		(layer "F.Cu")
@@
 	)
 	(segment
-		(start 143 65.86)
-		(end 140.785 68.075)
+		(start 111.675 55.325)
+		(end 113.75 53.25)
 		(width 0.2)
 		(layer "F.Cu")
@@
 	)
 	(segment
+		(start 142.75 53.25)
+		(end 143 53.5)
+		(width 0.2)
+		(layer "F.Cu")
+		(net "+3V3")
+	)
+	(segment
+		(start 104.075 55.53)
+		(end 106.545 58)
+		(width 0.2)
+		(layer "F.Cu")
+		(net "Net-(U4-A0)")
+	)
+	(segment
+		(start 113 61.055)
+		(end 113.05 61.105)
+		(width 0.2)
+		(layer "F.Cu")
+		(net "Net-(U4-A0)")
+	)
+	(segment
+		(start 114.625 55.375)
+		(end 117.925 55.375)
+		(width 0.2)
+		(layer "F.Cu")
+		(net "Net-(U4-A0)")
+	)
+	(segment
+		(start 113 58)
+		(end 113 61.055)
+		(width 0.2)
+		(layer "F.Cu")
+		(net "Net-(U4-A0)")
+	)
+	(segment
+		(start 106.545 58)
+		(end 113 58)
+		(width 0.2)
+		(layer "F.Cu")
+		(net "Net-(U4-A0)")
+	)
+	(segment
+		(start 113 61.055)
+		(end 113 57)
+		(width 0.2)
+		(layer "F.Cu")
+		(net "Net-(U4-A0)")
+	)
+	(segment
+		(start 113 57)
+		(end 114.625 55.375)
+		(width 0.2)
+		(layer "F.Cu")
+		(net "Net-(U4-A0)")
+	)
+	(segment
 		(start 65.31 61.81)
 		(end 60.805 61.81)
@@
 		(net "Net-(J1-CC1)")
 	)
-	(segment
-		(start 104.075 55.53)
-		(end 106.545 58)
-		(width 0.2)
-		(layer "F.Cu")
-		(net "Net-(U4-A0)")
-	)
-	(segment
-		(start 113 61.055)
-		(end 113.05 61.105)
-		(width 0.2)
-		(layer "F.Cu")
-		(net "Net-(U4-A0)")
-	)
-	(segment
-		(start 114.625 55.375)
-		(end 117.925 55.375)
-		(width 0.2)
-		(layer "F.Cu")
-		(net "Net-(U4-A0)")
-	)
-	(segment
-		(start 113 58)
-		(end 113 61.055)
-		(width 0.2)
-		(layer "F.Cu")
-		(net "Net-(U4-A0)")
-	)
-	(segment
-		(start 106.545 58)
-		(end 113 58)
-		(width 0.2)
-		(layer "F.Cu")
-		(net "Net-(U4-A0)")
-	)
-	(segment
-		(start 113 61.055)
-		(end 113 57)
-		(width 0.2)
-		(layer "F.Cu")
-		(net "Net-(U4-A0)")
-	)
-	(segment
-		(start 113 57)
-		(end 114.625 55.375)
-		(width 0.2)
-		(layer "F.Cu")
-		(net "Net-(U4-A0)")
-	)
 	(zone
 		(net "GND")
@@
 		(polygon
 			(pts
-				(xy 54 54) (xy 53 147) (xy 147 147) (xy 147 54)
+				(xy 54 54) (xy 53.005376 146.5) (xy 147 146.5) (xy 147 54)
 			)
 		)
